File: CNC Boosterpack.kicad_pcb (KiCad board)
At the start: 2 copper layers, 151.4 x 45.7 mm, 159 parts, among them J1 0, J10 Mist, J11 Flood, J12 StepperDrv, J13 StepperDrv, J14 StepperDrv, J15 5V off, J2 0, J3 0, J4 0, J5 0, J6 UART/GPIO, J7 I2C, J8 RESET, J9 Spindle, P1 Control, P2 Limits, P5 BPConnL, P6 BPConnR, Q1 MMBT5551, Q10 AO3400A, Q11 HSU3016, Q12 AO3400A, Q13 AO3400A, Q14 AO3400A, Q15 HSU3016, Q2 MMBT5551, Q3 MMBT5551, Q4 MMBT5551, Q5 MMBT5551, Q6 MMBT5551, Q7 MMBT5551, Q8 MMBT5551, Q9 MMBT5551, U1 TCA9406, U10 EL357N(B), U11 EL357N(B), U12 EL357N(B), U13 EL357N(B), U14 EL357N(B), U15 TPS54331DR, U2 M24C64, U3 EL357N(B), U4 EL357N(B), U5 EL357N(B), U6 EL357N(B), U7 EL357N(B), U8 EL357N(B), U9 EL357N(B)

Commit message: doc
Parts:
- P5, P6: moved to B.Cu
- moved J15 13.5 mm to (154.6, 135.5)
- moved C16 10.3 mm to (150.7, 138.7), turned to 180 degrees
- moved R64 9.06 mm to (150.7, 141.0)
- moved C15 8.51 mm to (157.5, 135.5), turned to 90 degrees
- moved J2 7.02 mm to (175.3, 120.0)
- moved C19 6.15 mm to (159.7, 140.7), turned to 90 degrees
- moved C14 4.34 mm to (160.5, 134.5), turned to 90 degrees
- moved R63 3.89 mm to (150.7, 143.2)
- moved C17 2.94 mm to (155.2, 145.5)
- moved J5 2.72 mm to (175.3, 117.3)
- moved C18 2.63 mm to (155.2, 148.5), turned to 180 degrees
- moved P6 2.54 mm to (167.6, 111.8), turned to 180 degrees
- moved P5 2.54 mm to (124.5, 111.8), turned to 180 degrees
- moved Lk5 0.76 mm to (86.2, 142.5)
- moved R62 0.61 mm to (155.2, 147.0)
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Connections:
- U15 pad 3: Net-(C19-Pad1) -> Net-(J15-Pad2)
- U15 pad 4: GND -> Net-(C16-Pad1)
- U15 pad 7: Net-(J15-Pad2) -> GND
- U15 pad 8: Net-(C16-Pad1) -> Net-(C19-Pad1)
Routing:
- net /STEPPER_EN_Z: track 72.9 -> 111.3 mm, vias 3 -> 1
- net /STEPPER_ALARM: track 107.5 -> 76.4 mm, vias 5 -> 2
- net +3.3V: track 254.7 -> 282.9 mm, vias 9 -> 14
- net /BP_SPINDLE_PWM: track 111.5 -> 138.4 mm, vias 2 -> 1
- net /STEPPER_EN_XY: track 63.4 -> 41.6 mm, vias 0 -> 4
- net GND: track 310.7 -> 330.4 mm, vias 216 -> 206
- net /BP_CS: track 35.4 -> 49.7 mm
- net /BP_Reset: track 51.1 -> 37.8 mm, vias 3 -> 2
- net /BP_FH: track 42.6 -> 55.0 mm
- net /BPR13: track 12.8 -> 23.0 mm, vias 2 -> 3
- net /STEPPER_X_DIR: track 84.7 -> 75.1 mm, vias 2 -> 3
- net /BP_SCL: track 38.1 -> 28.8 mm
- net /BP_SPINDLE_DIR: track 13.4 -> 22.4 mm, vias 0 -> 1
- net /BP_SPINDLE_EN: track 22.6 -> 31.5 mm, vias 2 -> 1
- net /VBUS: track 278.0 -> 270.2 mm, vias 16 -> 18
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Other:
- board text added: "(remove Q10 when populating Q11)"
- board text added: "(remove Q14 when populating Q15)"
- board text added: "+"
- board text added: "-"
- board text added: "- G - PWM DIR + EN +"
- board text added: "Fld"
- board text added: "GRBLhal Boosterpack ${ISSUE_DATE} by Sönke Peters Revision ${REVISION}"
- board text removed: "- G - PWM + DIR + EN"
- board text removed: "GRBLhal Boosterpack 2022-11-23 by Sönke Peters"
