File: CNC Boosterpack.kicad_sch (KiCad schematic)
At the start: 28 parts, among them J1 0, J10 Mist, J11 Flood, J2 0, J3 0, J4 0, J5 0, J6 UART/GPIO, J7 I2C, J8 RESET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

Commit message: some part rotations, JLCPCB ordered #W202211241441380
Parts:
- U1, U2: JLCPCB Rotation Offset (none) -> 90
Changed lines of the file:
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@@
+      (effects (font (size 1.27 1.27)) hide)
+    )
+    (property "JLCPCB Rotation Offset" "90" (id 5) (at 180.34 123.19 0)
       (effects (font (size 1.27 1.27)) hide)
     )
@@
       (effects (font (size 1.27 1.27)) hide)
     )
+    (property "JLCPCB Rotation Offset" "90" (id 5) (at 146.05 121.92 0)
+      (effects (font (size 1.27 1.27)) hide)
+    )

Commit message: doc
Parts:
- U1, U2: JLCPCB Rotation Offset 90 -> -90
Changed lines of the file:
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@@
   (title_block
     (title "GRBLhal Boosterpack")
-    (date "2022-11-23")
-    (rev "1.0")
-    (comment 1 "ruined by Sönke Peters")
+    (date "2022-12-20")
+    (rev "1.2")
+    (comment 1 "by Sönke Peters")
     (comment 2 "based on work by Terje Io and Expatria Technologies")
     (comment 4 "Licensed under CERN OHL v.1.2 or later")
@@
       (effects (font (size 1.27 1.27)) hide)
     )
-    (property "JLCPCB Rotation Offset" "90" (id 5) (at 180.34 123.19 0)
+    (property "JLCPCB Rotation Offset" "-90" (id 5) (at 180.34 123.19 0)
       (effects (font (size 1.27 1.27)) hide)
     )
@@
       (effects (font (size 1.27 1.27)) hide)
     )
-    (property "JLCPCB Rotation Offset" "90" (id 5) (at 146.05 121.92 0)
-      (effects (font (size 1.27 1.27)) hide)
-    )
+    (property "JLCPCB Rotation Offset" "-90" (id 5) (at 146.05 121.92 0)
+      (effects (font (size 1.27 1.27)) hide)
+    )
