File: mosfet_2possibilities.kicad_sch (KiCad schematic)
At the start: 9 parts, among them Q14 AO3400A, Q15 HSU3016, U14 EL357N(B)

Commit message: some part rotations, JLCPCB ordered #W202211241441380
Parts:
- Q14: JLCPCB Rotation Offset (none) -> 180
Changed lines of the file:
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@@
+      (effects (font (size 1.27 1.27)) hide)
+    )
+    (property "JLCPCB Rotation Offset" "180" (id 5) (at 143.51 102.87 0)
       (effects (font (size 1.27 1.27)) hide)
     )
