File: powersupply5v.kicad_sch (KiCad schematic)
At the start: 16 parts, among them J15 5V off, U15 TPS54331DR

Commit message: some part rotations, JLCPCB ordered #W202211241441380
Parts:
- C17: JLCPCB C32949 -> (none); JLCPCB Part # (none) -> C32949
- C18: JLCPCB C1542 -> (none); JLCPCB Part # (none) -> C1542
- R62: JLCPCB C25794 -> (none); JLCPCB Part # (none) -> C25794
Changed lines of the file:
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@@
       (effects (font (size 1.27 1.27)) hide)
     )
-    (property "JLCPCB" "C1542" (id 4) (at 124.46 106.68 0)
+    (property "JLCPCB Part #" "C1542" (id 4) (at 124.46 106.68 0)
       (effects (font (size 1.27 1.27)) hide)
     )
@@
       (effects (font (size 1.27 1.27)) hide)
     )
-    (property "JLCPCB" "C32949" (id 4) (at 114.3 106.68 0)
+    (property "JLCPCB Part #" "C32949" (id 4) (at 114.3 106.68 0)
       (effects (font (size 1.27 1.27)) hide)
     )
@@
       (effects (font (size 1.27 1.27)) hide)
     )
-    (property "JLCPCB" "C25794" (id 4) (at 124.46 99.06 0)
-      (effects (font (size 1.27 1.27)) hide)
-    )
+    (property "JLCPCB Part #" "C25794" (id 4) (at 124.46 99.06 0)
+      (effects (font (size 1.27 1.27)) hide)
+    )

Commit message: doc
Parts:
- L1: JLCPCB Rotation Offset (none) -> 180
- U15: symbol Regulator_Switching:TPS54336ADDA -> Library:TPS54331; JLCPCB Rotation Offset (none) -> -90
Connections:
- net GND: now also U15.7 (GND); no longer U15.4 (GND)
- net at J15.2 (Pin_2): now also U15.3 (EN); no longer U15.7 (EN)
- net at C16.1: now also U15.4 (SS); no longer U15.8 (SS)
- net at C19.1, D17.1 (K), L1.1: now also U15.8 (PH); no longer U15.3 (PH)
Changed lines of the file:
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@@
   (title_block
     (title "GRBLhal Boosterpack")
-    (date "2022-11-23")
-    (rev "1.0")
-    (comment 1 "ruined by Sönke Peters")
+    (date "2022-12-20")
+    (rev "1.2")
+    (comment 1 "by Sönke Peters")
     (comment 2 "based on work by Terje Io and Expatria Technologies")
     (comment 4 "Licensed under CERN OHL v.1.2 or later")
@@
     (stroke (width 0) (type default) (color 0 0 0 0))
   )
-  (wire (pts (xy 137.16 97.79) (xy 139.7 97.79))
+  (wire (pts (xy 137.16 97.79) (xy 140.335 97.79))
     (stroke (width 0) (type default) (color 0 0 0 0))
   )
@@
     (pin "2")
   )
-  (symbol (lib_id "Regulator_Switching:TPS54336ADDA") (at 139.7 87.63 0) (unit 1)
+  (symbol (lib_id "Library:TPS54331") (at 139.7 87.63 0) (unit 1)
     (in_bom yes) (on_board yes) (fields_autoplaced)
     (property "Reference" "U15" (id 0) (at 139.7 74.93 0))
     (property "Value" "TPS54331DR" (id 1) (at 139.7 77.47 0))
-    (property "Footprint" "Package_SO:TI_SO-PowerPAD-8_ThermalVias" (id 2) (at 162.56 96.52 0)
-      (effects (font (size 1.27 1.27)) hide)
-    )
-    (property "Datasheet" "https://www.ti.com/en/lit/gpn/tps54331" (id 3) (at 165.1 99.06 0)
+    (property "Footprint" "Package_SO:TI_SO-PowerPAD-8_ThermalVias" (id 2) (at 139.7 87.63 0)
+      (effects (font (size 1.27 1.27)) hide)
+    )
+    (property "Datasheet" "https://www.ti.com/en/lit/gpn/tps54331" (id 3) (at 139.7 87.63 0)
       (effects (font (size 1.27 1.27)) hide)
     )
     (property "JLCPCB Part #" "C9865" (id 4) (at 139.7 87.63 0)
+      (effects (font (size 1.27 1.27)) hide)
+    )
+    (property "JLCPCB Rotation Offset" "-90" (id 5) (at 139.7 87.63 0)
       (effects (font (size 1.27 1.27)) hide)
     )
@@
       (effects (font (size 1.27 1.27)) hide)
     )
+    (property "JLCPCB Rotation Offset" "180" (id 5) (at 176.53 87.63 90)
+      (effects (font (size 1.27 1.27)) hide)
+    )
